Commit message: Adding MoveIt Pro support

File: eli_cs_robot_description/urdf/cs.urdf.xacro (robot description, xacro)
@@ -2,5 +2,5 @@
 <robot xmlns:xacro="http://wiki.ros.org/xacro" name="$(arg name)">
    <!-- robot name parameter -->
-   <xacro:arg name="name" default="cs"/>
+   <xacro:arg name="name" default="cs612"/>
    <!-- import main macro -->
    <xacro:include filename="$(find eli_cs_robot_description)/urdf/cs_macro.xacro"/>
@@ -21,7 +21,7 @@
    <xacro:arg name="headless_mode" default="false" />
    <xacro:arg name="robot_ip" default="0.0.0.0" />
-   <xacro:arg name="script_filename" default=""/>
-   <xacro:arg name="output_recipe_filename" default=""/>
-   <xacro:arg name="input_recipe_filename" default=""/>
+   <xacro:arg name="script_filename" default="$(find eli_cs_robot_driver)/resources/external_control.script"/>
+   <xacro:arg name="output_recipe_filename" default="$(find eli_cs_robot_driver)/resources/input_recipe.txt"/>
+   <xacro:arg name="input_recipe_filename" default="$(find eli_cs_robot_driver)/resources/output_recipe.txt"/>
    <xacro:arg name="local_ip" default="0.0.0.0"/>
    <xacro:arg name="script_command_port" default="50004"/>

File: eli_cs_robot_moveit_config/srdf/cs.srdf.xacro (robot description, xacro)
@@ -2,5 +2,5 @@
 <robot xmlns:xacro="http://wiki.ros.org/xacro" name="$(arg name)">
   <!-- robot name parameter -->
-  <xacro:arg name="name" default="cs"/>
+  <xacro:arg name="name" default="cs612"/>
   <!-- parameters -->
   <xacro:arg name="prefix" default="" />

File: eli_cs_robot_moveit_config/srdf/cs_macro.srdf.xacro (robot description, xacro)
@@ -14,4 +14,8 @@
       <chain base_link="${prefix}base_link" tip_link="${prefix}tool0" />
     </group>
+    <group name="gripper">
+      <link name="${prefix}tool0" />
+    </group>
+    <end_effector name="gripper" parent_link="${prefix}flange" group="gripper" parent_group="${prefix}${name}_manipulator"/>
     <!--GROUP STATES - Purpose - Define a named state for a particular group, in terms of joint values. This is useful to define states like 'folded arms'-->
     <group_state name="${prefix}home" group="${prefix}${name}_manipulator">

Commit message: Update URDF and launch file for adjustable mounting point

File: eli_cs_robot_description/urdf/cs.urdf.xacro (robot description, xacro)
@@ -10,4 +10,5 @@
    <!-- parameters -->
    <xacro:arg name="tf_prefix" default="" />
+   <xacro:arg name="parent" default="world" />
    <xacro:arg name="joint_limit_params" default="$(find eli_cs_robot_description)/config/$(arg cs_type)/joint_limits.yaml"/>
    <xacro:arg name="kinematics_params" default="$(find eli_cs_robot_description)/config/$(arg cs_type)/default_kinematics.yaml"/>
@@ -46,11 +47,15 @@
    <!-- convert to property to use substitution in function -->
    <xacro:property name="initial_positions_file" default="$(arg initial_positions_file)"/>
-   <!-- create link fixed to the "world" -->
-   <link name="world" />
+   <!-- Convert argument into a Xacro variable -->
+   <xacro:property name="parent_var" value="$(arg parent)" />
+   <xacro:if value="${parent_var == 'world'}">
+     <!-- create link fixed to the "world" -->
+     <link name="world" />
+   </xacro:if>
    <!-- arm -->
    <xacro:cs_robot
      name="$(arg name)"
      tf_prefix="$(arg tf_prefix)"
-     parent="world"
+     parent="$(arg parent)"
      joint_limits_parameters_file="$(arg joint_limit_params)"
      kinematics_parameters_file="$(arg kinematics_params)"
@@ -83,5 +88,5 @@
      trajectory_port="$(arg trajectory_port)"
      >
-     <origin xyz="0 0 0" rpy="0 0 0" />          <!-- position robot in the world -->
+     <origin xyz="0 0 0" rpy="0 0 0" />          <!-- position robot in the parent_frame -->
    </xacro:cs_robot>
    <xacro:if value="$(arg sim_gazebo)">
