Commit message: fix: Driver startup crash
- Refactor to remove network connections from constructors and afford connection retries
- Incorporated changes and fixes from PickNik engagement

File: eli_cs_robot_description/urdf/cs.ros2_control.xacro (robot description, xacro)
@@ -13,4 +13,5 @@
     input_recipe_filename
     tf_prefix
+    robot_connect_timeout:=10
     robot_ip
     tool_voltage:=0
@@ -49,4 +50,5 @@
           <param name="trajectory_port">${trajectory_port}</param>
           <param name="tf_prefix">${tf_prefix}</param>
+          <param name="robot_connect_timeout">${robot_connect_timeout}</param>
           <param name="servoj_gain">2000</param>
           <param name="servoj_lookahead_time">0.08</param>

File: eli_cs_robot_description/urdf/cs.urdf.xacro (robot description, xacro)
@@ -21,4 +21,5 @@
    <!-- ros2_control related parameters -->
    <xacro:arg name="headless_mode" default="false" />
+   <xacro:arg name="robot_connect_timeout" default="10" />
    <xacro:arg name="robot_ip" default="0.0.0.0" />
    <xacro:arg name="script_filename" default="$(find eli_cs_robot_driver)/resources/external_control.script"/>
@@ -79,4 +80,5 @@
      tool_tcp_port="$(arg tool_tcp_port)"
      robot_ip="$(arg robot_ip)"
+     robot_connect_timeout="$(arg robot_connect_timeout)"
      script_filename="$(arg script_filename)"
      output_recipe_filename="$(arg output_recipe_filename)"

File: eli_cs_robot_description/urdf/cs_macro.xacro (robot description, xacro)
@@ -46,4 +46,5 @@
     tool_tcp_port:=54321
     robot_ip:=0.0.0.0
+    robot_connect_timeout:=10
     script_filename:=to_be_filled_by_cs_robot_driver
     output_recipe_filename:=to_be_filled_by_cs_robot_driver
@@ -79,4 +80,5 @@
         tf_prefix="${tf_prefix}"
         robot_ip="${robot_ip}"
+        robot_connect_timeout="${robot_connect_timeout}"
         use_tool_communication="${use_tool_communication}"
         tool_voltage="${tool_voltage}"
@@ -202,9 +204,15 @@
       <xacro:build_inertial mass="${wrist_3_mass}" cog="${prop_wrist_3_cog}" inertia="${prop_wrist_3_inertia}"/>
     </link>
-    <!-- base_joint fixes base_link to the environment -->
+    <link name="fts_link" />
+    <joint name="fts_link_joint" type="fixed">
+      <parent link="${parent}" />
+      <child link="fts_link" />
+      <origin xyz="0.0 0 0.0" rpy="3.14 0 3.14" />
+    </joint>
+     <!-- base_joint fixes base_link to the environment -->
     <joint name="${tf_prefix}base_joint" type="fixed">
-      <xacro:insert_block name="origin" />
-      <parent link="${parent}" />
+      <parent link="fts_link" />
       <child link="${tf_prefix}base_link" />
+      <origin xyz="0.0 0 0.0" rpy="-3.14 0 -3.14" />
     </joint>
     <!-- joints - main serial chain -->

Commit message: Merge latest Elite driver + free drive fix

File: eli_cs_robot_description/urdf/cs.ros2_control.xacro (robot description, xacro)
@@ -284,4 +284,9 @@
           <command_interface name="zero_ftsensor_async_success"/>
         </gpio>
+        <gpio name="${tf_prefix}freedrive_mode">
+          <command_interface name="freedrive_async_success"/>
+          <command_interface name="freedrive_start_cmd"/>
+          <command_interface name="freedrive_end_cmd"/>
+        </gpio>
         <gpio name="${tf_prefix}system_interface">
           <state_interface name="initialized"/>

File: eli_cs_robot_description/urdf/cs.urdf.xacro (robot description, xacro)
@@ -10,5 +10,4 @@
    <!-- parameters -->
    <xacro:arg name="tf_prefix" default="" />
-   <xacro:arg name="parent" default="world" />
    <xacro:arg name="joint_limit_params" default="$(find eli_cs_robot_description)/config/$(arg cs_type)/joint_limits.yaml"/>
    <xacro:arg name="kinematics_params" default="$(find eli_cs_robot_description)/config/$(arg cs_type)/default_kinematics.yaml"/>
@@ -23,7 +22,7 @@
    <xacro:arg name="robot_connect_timeout" default="10" />
    <xacro:arg name="robot_ip" default="0.0.0.0" />
-   <xacro:arg name="script_filename" default="$(find eli_cs_robot_driver)/resources/external_control.script"/>
-   <xacro:arg name="output_recipe_filename" default="$(find eli_cs_robot_driver)/resources/input_recipe.txt"/>
-   <xacro:arg name="input_recipe_filename" default="$(find eli_cs_robot_driver)/resources/output_recipe.txt"/>
+   <xacro:arg name="script_filename" default=""/>
+   <xacro:arg name="output_recipe_filename" default=""/>
+   <xacro:arg name="input_recipe_filename" default=""/>
    <xacro:arg name="local_ip" default="0.0.0.0"/>
    <xacro:arg name="script_command_port" default="50004"/>
@@ -48,15 +47,11 @@
    <!-- convert to property to use substitution in function -->
    <xacro:property name="initial_positions_file" default="$(arg initial_positions_file)"/>
-   <!-- Convert argument into a Xacro variable -->
-   <xacro:property name="parent_var" value="$(arg parent)" />
-   <xacro:if value="${parent_var == 'world'}">
-     <!-- create link fixed to the "world" -->
-     <link name="world" />
-   </xacro:if>
+   <!-- create link fixed to the "world" -->
+   <link name="world" />
    <!-- arm -->
    <xacro:cs_robot
      name="$(arg name)"
      tf_prefix="$(arg tf_prefix)"
-     parent="$(arg parent)"
+     parent="world"
      joint_limits_parameters_file="$(arg joint_limit_params)"
      kinematics_parameters_file="$(arg kinematics_params)"
@@ -90,5 +85,5 @@
      trajectory_port="$(arg trajectory_port)"
      >
-     <origin xyz="0 0 0" rpy="0 0 0" />          <!-- position robot in the parent_frame -->
+     <origin xyz="0 0 0" rpy="0 0 0" />          <!-- position robot in the world -->
    </xacro:cs_robot>
    <xacro:if value="$(arg sim_gazebo)">

File: eli_cs_robot_description/urdf/cs_macro.xacro (robot description, xacro)
@@ -204,15 +204,9 @@
       <xacro:build_inertial mass="${wrist_3_mass}" cog="${prop_wrist_3_cog}" inertia="${prop_wrist_3_inertia}"/>
     </link>
-    <link name="fts_link" />
-    <joint name="fts_link_joint" type="fixed">
-      <parent link="${parent}" />
-      <child link="fts_link" />
-      <origin xyz="0.0 0 0.0" rpy="3.14 0 3.14" />
-    </joint>
      <!-- base_joint fixes base_link to the environment -->
     <joint name="${tf_prefix}base_joint" type="fixed">
-      <parent link="fts_link" />
+      <xacro:insert_block name="origin" />
+      <parent link="${parent}" />
       <child link="${tf_prefix}base_link" />
-      <origin xyz="0.0 0 0.0" rpy="-3.14 0 -3.14" />
     </joint>
     <!-- joints - main serial chain -->
