Commit message: Update SRDF to have configurable root link

File: eli_cs_robot_moveit_config/srdf/cs.srdf.xacro (robot description, xacro)
@@ -5,5 +5,6 @@
   <!-- parameters -->
   <xacro:arg name="prefix" default="" />
+  <xacro:arg name="manipulator_group_base_link" default="base_link" />
   <xacro:include filename="$(find eli_cs_robot_moveit_config)/srdf/cs_macro.srdf.xacro"/>
-  <xacro:cs_srdf name="$(arg name)" prefix="$(arg prefix)"/>
+  <xacro:cs_srdf name="$(arg name)" prefix="$(arg prefix)" manipulator_group_base_link="$(arg manipulator_group_base_link)"/>
 </robot>

File: eli_cs_robot_moveit_config/srdf/cs_macro.srdf.xacro (robot description, xacro)
@@ -5,5 +5,5 @@
     A URDF file must exist for this robot as well, where the joints and the links that are referenced are defined
 -->
-  <xacro:macro name="cs_srdf" params="name prefix">
+  <xacro:macro name="cs_srdf" params="name prefix manipulator_group_base_link">
     <!--GROUPS - Representation of a set of joints and links. This can be useful for specifying DOF to plan for, defining arms, end effectors, etc-->
     <!--LINKS - When a link is specified, the parent joint of that link (if it exists) is automatically included-->
@@ -12,4 +12,7 @@
     <!--SUBGROUPS - Groups can also be formed by referencing to already defined group names-->
     <group name="${prefix}${name}_manipulator">
+      <chain base_link="${prefix}${manipulator_group_base_link}" tip_link="${prefix}tool0" />
+    </group>
+    <group name="${prefix}${name}_manipulator_arm">
       <chain base_link="${prefix}base_link" tip_link="${prefix}tool0" />
     </group>
